Commit message: Release Locomotion Beyond Feet
Introduces the Locomotion Beyond Feet system, enabling ToddlerBot to perform complex locomotion skills beyond standard walking.

Key additions:
- Multi-skill locomotion: climbing (walls, boxes, stairs) and crawling
- Depth data collection pipeline for training and evaluation
- Vision-based skill classifier for locomotion mode selection
- Policy switching and chaining across locomotion skills
- Terrain generation with elevation mapping
- Motion reference library for diverse locomotion modes
- Expanded keyframe motions and RL training environments

File: toddlerbot/descriptions/toddlerbot_2xc/toddlerbot_2xc.urdf (robot description, URDF)
Before this commit: robot toddlerbot_2xc, 91 links, 90 joints
Links:
- link left_ankle_roll_link: geometry collision box size=0.11 0.042 0.014 type=box; visual mesh filename=assets/left_ankle_roll_link_visual.stl scale=1.0 1.0 1.0
- link right_ankle_roll_link: geometry collision box size=0.11 0.042 0.014 type=box; visual mesh filename=assets/right_ankle_roll_link_visual.stl scale=1.0 1.0 1.0

File: toddlerbot/descriptions/toddlerbot_2xm/toddlerbot_2xm.urdf (robot description, URDF)
Before this commit: robot toddlerbot_2xm, 91 links, 90 joints
Links:
- link left_ankle_roll_link: geometry collision box size=0.11 0.042 0.014 type=box; visual mesh filename=assets/left_ankle_roll_link_visual.stl scale=1.0 1.0 1.0
- link right_ankle_roll_link: geometry collision box size=0.11 0.042 0.014 type=box; visual mesh filename=assets/right_ankle_roll_link_visual.stl scale=1.0 1.0 1.0
